File: PCB/Bike_Speedo.sch (EAGLE design)
At the start: 29 parts, among them IC2 TPS61202, J1 TE_CONNECTIVITY_1981568-1TE_C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, P1 BAT, U1 MICROCHIP_MCP73833-AMI-UNMICR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

Commit message: Update schematic
Parts:
- removed C11: 100nF, rcl:C-EUC0805
- removed IC1, IC3: (no value), arduino:ARDUINO2009_PIN_22
- added C13, C14: 100nF, rcl:C-EUC0805
- added LCD: (no value), arduino:ARDUINO2009_PIN_22
- added U2: NUCLEO-F446RE, NUCLEO-F446RE:NUCLEO-F446RE
- R1, R2, R3: value 470R -> 1k
Connections:
- removed net N$1: IC1G$1.(SS)PB2, IC3G$1.(SS)PB2
- removed net N$13: IC1G$1.(MISO)PB4, IC3G$1.(MISO)PB4
- removed net N$16: IC1G$1.(SCK)PB5, IC3G$1.(SCK)PB5
- removed net N$17: IC1G$1.(OC1)PB1, IC3G$1.(OC1)PB1
- removed net N$18: IC1G$1.(ICP)PB0, IC3G$1.(ICP)PB0
- removed net N$19: IC1G$1.(AIN1)PD7, IC3G$1.(AIN1)PD7
- removed net N$20: IC1G$1.(AIN0)PD6, IC3G$1.(AIN0)PD6
- removed net N$21: IC1G$1.(T1)PD5, IC3G$1.(T1)PD5
- removed net N$22: IC1G$1.(T0)PD4, IC3G$1.(T0)PD4
- removed net N$23: IC1G$1.(INT1)PD3, IC3G$1.(INT1)PD3
- removed net N$24: IC1G$1.!RESET, IC3G$1.!RESET
- removed net N$5: IC1G$1.(MOSI)PB3, IC3G$1.(MOSI)PB3
- new net LCD_BL: LCDG$1.(OC1)PB1, U2G$6.D9
- new net LCD_CS: LCDG$1.(SS)PB2, U2G$6.D10
- new net LCD_DC: LCDG$1.(AIN1)PD7, U2G$4.D7
- new net LCD_RST: LCDG$1.(ICP)PB0, U2G$6.D8
- new net MISO: LCDG$1.(MISO)PB4, U2G$6.D12
- new net MOSI: LCDG$1.(MOSI)PB3, U2G$6.D11
- new net RESET: LCDG$1.!RESET, U2G$1.CN7_RESET, U2G$3.CN6_RESET
- new net SCLK: LCDG$1.(SCK)PB5, U2G$6.D13
- new net TP_BUSY: LCDG$1.(AIN0)PD6, U2G$4.D6
- new net TP_CS: LCDG$1.(T0)PD4, U2G$4.D4
- new net TP_IRQ: LCDG$1.(INT1)PD3, U2G$4.D3
- net +5V: now also C13.1, C14.2, LCDG$2.+5V, U2G$1.CN7_+5V, U2G$1.E5V, U2G$3.CN6_+5V; no longer C11.2, IC1G$4.+VIN, IC3G$2.+5V
- net GND: now also C13.2, C14.1, LCDG$2.GND, U2G$1.CN7_GND, U2G$2.CN10_GND, U2G$3.CN6_GND, U2G$6.CN5_GND; no longer C11.1, IC1G$4.GND, IC3G$2.GND
- net SIGNAL_SENSOR: now also U2G$2.PC9
Other:
- moved on the sheet: C12, SV1

Commit message: update PCB
Parts:
- removed C12: 100nF, rcl:C-EUC0805
- removed LCD: (no value), arduino:ARDUINO2009_PIN_22
- C3: value 100nD -> 100nF
Connections:
- net +5V: no longer C12.2, LCDG$2.+5V
- net GND: no longer C12.1, LCDG$2.GND
- net LCD_BL: no longer LCDG$1.(OC1)PB1
- net LCD_CS: no longer LCDG$1.(SS)PB2
- net LCD_DC: no longer LCDG$1.(AIN1)PD7
- net LCD_RST: no longer LCDG$1.(ICP)PB0
- net MISO: no longer LCDG$1.(MISO)PB4
- net MOSI: no longer LCDG$1.(MOSI)PB3
- net RESET: no longer LCDG$1.!RESET, U2G$1.CN7_RESET
- net SCLK: no longer LCDG$1.(SCK)PB5
- net TP_BUSY: no longer LCDG$1.(AIN0)PD6
- net TP_CS: no longer LCDG$1.(T0)PD4
- net TP_IRQ: no longer LCDG$1.(INT1)PD3
Changed lines of the file:
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@@
 <layers>
 <layer number="1" name="Top" color="4" fill="1" visible="no" active="no"/>
+<layer number="2" name="Route2" color="1" fill="3" visible="no" active="no"/>
+<layer number="3" name="Route3" color="4" fill="3" visible="no" active="no"/>
+<layer number="4" name="Route4" color="1" fill="4" visible="no" active="no"/>
+<layer number="5" name="Route5" color="4" fill="4" visible="no" active="no"/>
+<layer number="6" name="Route6" color="1" fill="8" visible="no" active="no"/>
+<layer number="7" name="Route7" color="4" fill="8" visible="no" active="no"/>
+<layer number="8" name="Route8" color="1" fill="2" visible="no" active="no"/>
+<layer number="9" name="Route9" color="4" fill="2" visible="no" active="no"/>
+<layer number="10" name="Route10" color="1" fill="7" visible="no" active="no"/>
+<layer number="11" name="Route11" color="4" fill="7" visible="no" active="no"/>
+<layer number="12" name="Route12" color="1" fill="5" visible="no" active="no"/>
+<layer number="13" name="Route13" color="4" fill="5" visible="no" active="no"/>
+<layer number="14" name="Route14" color="1" fill="6" visible="no" active="no"/>
+<layer number="15" name="Route15" color="4" fill="6" visible="no" active="no"/>
 <layer number="16" name="Bottom" color="1" fill="1" visible="no" active="no"/>
 <layer number="17" name="Pads" color="2" fill="1" visible="no" active="no"/>
@@
 <part name="SUPPLY3" library="supply2" library_urn="urn:adsk.eagle:library:372" deviceset="GND" device=""/>
 <part name="SUPPLY4" library="supply2" library_urn="urn:adsk.eagle:library:372" deviceset="GND" device=""/>
-<part name="C3" library="rcl" library_urn="urn:adsk.eagle:library:334" deviceset="C-EU" device="C0805" package3d_urn="urn:adsk.eagle:package:23617/2" value="100nD"/>
+<part name="C3" library="rcl" library_urn="urn:adsk.eagle:library:334" deviceset="C-EU" device="C0805" package3d_urn="urn:adsk.eagle:package:23617/2" value="100nF"/>
 <part name="C4" library="rcl" library_urn="urn:adsk.eagle:library:334" deviceset="C-EU" device="C0805" package3d_urn="urn:adsk.eagle:package:23617/2" value="10uF"/>
 <part name="C5" library="rcl" library_urn="urn:adsk.eagle:library:334" deviceset="C-EU" device="C0805" package3d_urn="urn:adsk.eagle:package:23617/2" value="1uF"/>
@@
 <part name="SUPPLY17" library="supply2" library_urn="urn:adsk.eagle:library:372" deviceset="GND" device=""/>
 <part name="S1" library="smd-special" library_urn="urn:adsk.eagle:library:362" deviceset="SWS001" device="" package3d_urn="urn:adsk.eagle:package:26467/1"/>
-<part name="LCD" library="arduino" deviceset="ARDUINO2009_PIN_2" device="2"/>
-<part name="SUPPLY19" library="supply2" library_urn="urn:adsk.eagle:library:372" deviceset="GND" device=""/>
-<part name="C12" library="rcl" library_urn="urn:adsk.eagle:library:334" deviceset="C-EU" device="C0805" package3d_urn="urn:adsk.eagle:package:23617/2" value="100nF"/>
 <part name="SV1" library="con-lstb" library_urn="urn:adsk.eagle:library:162" deviceset="MA03-1" device="" package3d_urn="urn:adsk.eagle:package:8339/1" value="SENSOR"/>
 <part name="SUPPLY20" library="supply2" library_urn="urn:adsk.eagle:library:372" deviceset="GND" device=""/>
@@
 <attribute name="NAME" x="185.42" y="162.56" size="1.778" layer="95" rot="R90"/>
 <attribute name="VALUE" x="192.405" y="162.56" size="1.778" layer="96" rot="R90"/>
-</instance>
-<instance part="LCD" gate="G$1" x="419.1" y="114.3" smashed="yes" rot="MR0">
-<attribute name="NAME" x="434.34" y="143.51" size="1.6764" layer="95" rot="MR0"/>
-</instance>
-<instance part="LCD" gate="G$2" x="414.02" y="58.42" smashed="yes"/>
-<instance part="SUPPLY19" gate="GND" x="414.02" y="43.18" smashed="yes">
-<attribute name="VALUE" x="412.115" y="40.005" size="1.778" layer="96"/>
-</instance>
-<instance part="C12" gate="G$1" x="426.72" y="58.42" smashed="yes" rot="R180">
-<attribute name="NAME" x="425.196" y="58.039" size="1.778" layer="95" rot="R180"/>
-<attribute name="VALUE" x="425.196" y="63.119" size="1.778" layer="96" rot="R180"/>
 </instance>
 <instance part="SV1" gate="G$1" x="248.92" y="91.44" smashed="yes" rot="R180">
@@
 </segment>
 <segment>
-<pinref part="LCD" gate="G$2" pin="GND"/>
-<wire x1="414.02" y1="48.26" x2="414.02" y2="45.72" width="0.1524" layer="91"/>
-<pinref part="SUPPLY19" gate="GND" pin="GND"/>
-<pinref part="C12" gate="G$1" pin="1"/>
-<wire x1="426.72" y1="55.88" x2="426.72" y2="48.26" width="0.1524" layer="91"/>
-<wire x1="426.72" y1="48.26" x2="414.02" y2="48.26" width="0.1524" layer="91"/>
-<junction x="414.02" y="48.26"/>
-</segment>
-<segment>
 <pinref part="SV1" gate="G$1" pin="2"/>
 <wire x1="241.3" y1="91.44" x2="236.22" y2="91.44" width="0.1524" layer="91"/>
@@
 <junction x="162.56" y="68.58"/>
 <label x="167.64" y="68.58" size="1.778" layer="95" xref="yes"/>
-</segment>
-<segment>
-<pinref part="LCD" gate="G$2" pin="+5V"/>
-<wire x1="414.02" y1="68.58" x2="414.02" y2="71.12" width="0.1524" layer="91"/>
-<label x="414.02" y="71.12" size="1.778" layer="95" rot="R90" xref="yes"/>
-<pinref part="C12" gate="G$1" pin="2"/>
-<wire x1="426.72" y1="63.5" x2="426.72" y2="68.58" width="0.1524" layer="91"/>
-<wire x1="426.72" y1="68.58" x2="414.02" y2="68.58" width="0.1524" layer="91"/>
-<junction x="414.02" y="68.58"/>
 </segment>
 <segment>
@@
 <net name="RESET" class="0">
 <segment>
-<pinref part="LCD" gate="G$1" pin="!RESET"/>
-<wire x1="439.42" y1="137.16" x2="444.5" y2="137.16" width="0.1524" layer="91"/>
-<label x="444.5" y="137.16" size="1.778" layer="95" xref="yes"/>
-</segment>
-<segment>
-<pinref part="U2" gate="G$1" pin="CN7_RESET"/>
-<wire x1="327.66" y1="60.96" x2="325.12" y2="60.96" width="0.1524" layer="91"/>
-<wire x1="325.12" y1="60.96" x2="325.12" y2="66.04" width="0.1524" layer="91"/>
-<label x="325.12" y="66.04" size="1.778" layer="95" rot="R90" xref="yes"/>
-</segment>
-<segment>
 <pinref part="U2" gate="G$3" pin="CN6_RESET"/>
 <wire x1="398.78" y1="10.16" x2="393.7" y2="10.16" width="0.1524" layer="91"/>
@@
 <net name="TP_IRQ" class="0">
 <segment>
-<pinref part="LCD" gate="G$1" pin="(INT1)PD3"/>
-<wire x1="398.78" y1="101.6" x2="396.24" y2="101.6" width="0.1524" layer="91"/>
-<label x="396.24" y="101.6" size="1.778" layer="95" rot="R180" xref="yes"/>
-</segment>
-<segment>
 <pinref part="U2" gate="G$4" pin="D3"/>
 <wire x1="314.96" y1="101.6" x2="332.74" y2="101.6" width="0.1524" layer="91"/>
@@
 <net name="TP_CS" class="0">
 <segment>
-<pinref part="LCD" gate="G$1" pin="(T0)PD4"/>
-<wire x1="398.78" y1="99.06" x2="381" y2="99.06" width="0.1524" layer="91"/>
-<label x="381" y="99.06" size="1.778" layer="95" rot="R180" xref="yes"/>
-</segment>
-<segment>
 <pinref part="U2" gate="G$4" pin="D4"/>
 <wire x1="314.96" y1="99.06" x2="317.5" y2="99.06" width="0.1524" layer="91"/>
@@
 <net name="TP_BUSY" class="0">
 <segment>
-<pinref part="LCD" gate="G$1" pin="(AIN0)PD6"/>
-<wire x1="398.78" y1="93.98" x2="396.24" y2="93.98" width="0.1524" layer="91"/>
-<label x="396.24" y="93.98" size="1.778" layer="95" rot="R180" xref="yes"/>
-</segment>
-<segment>
 <pinref part="U2" gate="G$4" pin="D6"/>
 <wire x1="314.96" y1="93.98" x2="332.74" y2="93.98" width="0.1524" layer="91"/>
@@
 <net name="LCD_DC" class="0">
 <segment>
-<pinref part="LCD" gate="G$1" pin="(AIN1)PD7"/>
-<wire x1="398.78" y1="91.44" x2="381" y2="91.44" width="0.1524" layer="91"/>
-<label x="381" y="91.44" size="1.778" layer="95" rot="R180" xref="yes"/>
-</segment>
-<segment>
 <pinref part="U2" gate="G$4" pin="D7"/>
 <wire x1="314.96" y1="91.44" x2="317.5" y2="91.44" width="0.1524" layer="91"/>
@@
 <net name="LCD_RST" class="0">
 <segment>
-<pinref part="LCD" gate="G$1" pin="(ICP)PB0"/>
-<wire x1="398.78" y1="137.16" x2="396.24" y2="137.16" width="0.1524" layer="91"/>
-<label x="396.24" y="137.16" size="1.778" layer="95" rot="R180" xref="yes"/>
-</segment>
-<segment>
 <pinref part="U2" gate="G$6" pin="D8"/>
 <wire x1="314.96" y1="147.32" x2="332.74" y2="147.32" width="0.1524" layer="91"/>
@@
 <net name="LCD_BL" class="0">
 <segment>
-<pinref part="LCD" gate="G$1" pin="(OC1)PB1"/>
-<wire x1="398.78" y1="134.62" x2="381" y2="134.62" width="0.1524" layer="91"/>
-<label x="381" y="134.62" size="1.778" layer="95" rot="R180" xref="yes"/>
-</segment>
-<segment>
 <pinref part="U2" gate="G$6" pin="D9"/>
 <wire x1="314.96" y1="144.78" x2="317.5" y2="144.78" width="0.1524" layer="91"/>
@@
 <net name="LCD_CS" class="0">
 <segment>
-<pinref part="LCD" gate="G$1" pin="(SS)PB2"/>
-<wire x1="398.78" y1="132.08" x2="396.24" y2="132.08" width="0.1524" layer="91"/>
-<label x="396.24" y="132.08" size="1.778" layer="95" rot="R180" xref="yes"/>
-</segment>
-<segment>
 <pinref part="U2" gate="G$6" pin="D10"/>
 <wire x1="314.96" y1="142.24" x2="332.74" y2="142.24" width="0.1524" layer="91"/>
@@
 <net name="MOSI" class="0">
 <segment>
-<pinref part="LCD" gate="G$1" pin="(MOSI)PB3"/>
-<wire x1="398.78" y1="129.54" x2="381" y2="129.54" width="0.1524" layer="91"/>
-<label x="381" y="129.54" size="1.778" layer="95" rot="R180" xref="yes"/>
-</segment>
-<segment>
 <pinref part="U2" gate="G$6" pin="D11"/>
 <wire x1="314.96" y1="139.7" x2="317.5" y2="139.7" width="0.1524" layer="91"/>
@@
 <net name="MISO" class="0">
 <segment>
-<pinref part="LCD" gate="G$1" pin="(MISO)PB4"/>
-<wire x1="398.78" y1="127" x2="396.24" y2="127" width="0.1524" layer="91"/>
-<label x="396.24" y="127" size="1.778" layer="95" rot="R180" xref="yes"/>
-</segment>
-<segment>
 <pinref part="U2" gate="G$6" pin="D12"/>
 <wire x1="314.96" y1="137.16" x2="332.74" y2="137.16" width="0.1524" layer="91"/>
@@
 <net name="SCLK" class="0">
 <segment>
-<pinref part="LCD" gate="G$1" pin="(SCK)PB5"/>
-<wire x1="398.78" y1="124.46" x2="381" y2="124.46" width="0.1524" layer="91"/>
-<label x="381" y="124.46" size="1.778" layer="95" rot="R180" xref="yes"/>
-</segment>
-<segment>
 <pinref part="U2" gate="G$6" pin="D13"/>

Commit message: modified PCB
Parts:
- added C11: 10pF, rcl:C-EUC0805
- added R6: 1Meg, rcl:R-EU_R0805
- added R7: (no value), ptc-ntc:PTC660
- added R8: 0R, rcl:R-EU_R0805
Connections:
- new net N$1: J1.VBUS, R7.1
- new net N$5: C11.2, J1.GND, J1.SHLD1, J1.SHLD2, J1.SHLD3, J1.SHLD4, J1.SHLD5, J1.SHLD6, R6.2
- net +5V: no longer U2G$1.CN7_+5V, U2G$3.CN6_+5V
- net GND: now also C11.1, R6.1, R8.1, R8.2; no longer J1.GND, J1.SHLD1, J1.SHLD2, J1.SHLD3, J1.SHLD4, J1.SHLD5, J1.SHLD6
- net N$4: now also R7.2; no longer J1.VBUS
Other:
- moved on the sheet: C13, C14, C3, J1, SV1, U2G$1, U2G$2, U2G$3, U2G$4, U2G$6

Commit message: Update schematic and board
Connections:
- removed net LCD_BL: U2G$6.D9
- removed net LCD_CS: U2G$6.D10
- removed net LCD_DC: U2G$4.D7
- removed net LCD_RST: U2G$6.D8
- removed net MISO: U2G$6.D12
- removed net MOSI: U2G$6.D11
- removed net RESET: U2G$3.CN6_RESET
- removed net SCLK: U2G$6.D13
- removed net TP_BUSY: U2G$4.D6
- removed net TP_CS: U2G$4.D4
- removed net TP_IRQ: U2G$4.D3
- net GND: no longer U2G$3.CN6_GND, U2G$6.CN5_GND
Other:
- moved on the sheet: R8
Changed lines of the file:
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@@
 <part name="SUPPLY20" library="supply2" library_urn="urn:adsk.eagle:library:372" deviceset="GND" device=""/>
 <part name="U2" library="NUCLEO-F446RE" deviceset="NUCLEO-F446RE" device=""/>
-<part name="SUPPLY21" library="supply2" library_urn="urn:adsk.eagle:library:372" deviceset="GND" device=""/>
 <part name="SUPPLY22" library="supply2" library_urn="urn:adsk.eagle:library:372" deviceset="GND" device=""/>
 <part name="C13" library="rcl" library_urn="urn:adsk.eagle:library:334" deviceset="C-EU" device="C0805" package3d_urn="urn:adsk.eagle:package:23617/2" value="100nF"/>
@@
 <part name="SUPPLY18" library="supply2" library_urn="urn:adsk.eagle:library:372" deviceset="GND" device=""/>
 <part name="SUPPLY19" library="supply2" library_urn="urn:adsk.eagle:library:372" deviceset="GND" device=""/>
-<part name="SUPPLY26" library="supply2" library_urn="urn:adsk.eagle:library:372" deviceset="GND" device=""/>
 </parts>
 <sheets>
@@
 <attribute name="VALUE" x="256.54" y="-1.27" size="1.778" layer="96" rot="R180"/>
 </instance>
-<instance part="U2" gate="G$4" x="251.46" y="99.06" smashed="yes" rot="MR0">
-<attribute name="NAME" x="256.54" y="113.03" size="1.778" layer="95" rot="MR0"/>
-<attribute name="VALUE" x="256.54" y="85.09" size="1.778" layer="96" rot="R180"/>
-</instance>
-<instance part="U2" gate="G$6" x="246.38" y="137.16" smashed="yes" rot="MR0">
-<attribute name="NAME" x="256.54" y="153.67" size="1.778" layer="95" rot="MR0"/>
-<attribute name="VALUE" x="256.54" y="118.11" size="1.778" layer="96" rot="R180"/>
-</instance>
-<instance part="SUPPLY21" gate="GND" x="228.6" y="116.84" smashed="yes">
-<attribute name="VALUE" x="226.695" y="113.665" size="1.778" layer="96"/>
-</instance>
 <instance part="SUPPLY22" gate="GND" x="223.52" y="-2.54" smashed="yes">
 <attribute name="VALUE" x="221.615" y="-5.715" size="1.778" layer="96"/>
@@
 <attribute name="VALUE" x="320.675" y="-10.795" size="1.778" layer="96"/>
 </instance>
-<instance part="U2" gate="G$3" x="365.76" y="10.16" smashed="yes">
-<attribute name="NAME" x="350.52" y="21.59" size="1.778" layer="95"/>
-<attribute name="VALUE" x="350.52" y="-3.81" size="1.778" layer="96" rot="MR180"/>
-</instance>
 <instance part="SUPPLY25" gate="GND" x="330.2" y="55.88" smashed="yes">
 <attribute name="VALUE" x="328.295" y="52.705" size="1.778" layer="96"/>
@@
 <attribute name="VALUE" x="35.433" y="155.448" size="1.778" layer="96" rot="R270"/>
 </instance>
-<instance part="R8" gate="G$1" x="177.8" y="45.72" smashed="yes" rot="R180">
-<attribute name="NAME" x="181.61" y="44.2214" size="1.778" layer="95" rot="R180"/>
-<attribute name="VALUE" x="181.61" y="49.022" size="1.778" layer="96" rot="R180"/>
-</instance>
-<instance part="SUPPLY18" gate="GND" x="185.42" y="40.64" smashed="yes">
-<attribute name="VALUE" x="183.515" y="37.465" size="1.778" layer="96"/>
-</instance>
-<instance part="SUPPLY19" gate="GND" x="170.18" y="40.64" smashed="yes">
-<attribute name="VALUE" x="168.275" y="37.465" size="1.778" layer="96"/>
-</instance>
-<instance part="SUPPLY26" gate="GND" x="388.62" y="-5.08" smashed="yes">
-<attribute name="VALUE" x="386.715" y="-8.255" size="1.778" layer="96"/>
+<instance part="R8" gate="G$1" x="182.88" y="38.1" smashed="yes" rot="R180">
+<attribute name="NAME" x="186.69" y="36.6014" size="1.778" layer="95" rot="R180"/>
+<attribute name="VALUE" x="186.69" y="41.402" size="1.778" layer="96" rot="R180"/>
+</instance>
+<instance part="SUPPLY18" gate="GND" x="190.5" y="33.02" smashed="yes">
+<attribute name="VALUE" x="188.595" y="29.845" size="1.778" layer="96"/>
+</instance>
+<instance part="SUPPLY19" gate="GND" x="175.26" y="33.02" smashed="yes">
+<attribute name="VALUE" x="173.355" y="29.845" size="1.778" layer="96"/>
 </instance>
 </instances>
@@
 </segment>
 <segment>
-<pinref part="U2" gate="G$6" pin="CN5_GND"/>
-<wire x1="231.14" y1="121.92" x2="228.6" y2="121.92" width="0.1524" layer="91"/>
-<pinref part="SUPPLY21" gate="GND" pin="GND"/>
-<wire x1="228.6" y1="121.92" x2="228.6" y2="119.38" width="0.1524" layer="91"/>
-</segment>
-<segment>
 <pinref part="U2" gate="G$2" pin="CN10_GND"/>
 <wire x1="226.06" y1="2.54" x2="223.52" y2="2.54" width="0.1524" layer="91"/>
@@
 <segment>
 <pinref part="SUPPLY19" gate="GND" pin="GND"/>
-<wire x1="170.18" y1="43.18" x2="170.18" y2="45.72" width="0.1524" layer="91"/>
+<wire x1="175.26" y1="35.56" x2="175.26" y2="38.1" width="0.1524" layer="91"/>
 <pinref part="R8" gate="G$1" pin="2"/>
-<wire x1="170.18" y1="45.72" x2="172.72" y2="45.72" width="0.1524" layer="91"/>
+<wire x1="175.26" y1="38.1" x2="177.8" y2="38.1" width="0.1524" layer="91"/>
 </segment>
 <segment>
 <pinref part="R8" gate="G$1" pin="1"/>
-<wire x1="182.88" y1="45.72" x2="185.42" y2="45.72" width="0.1524" layer="91"/>
+<wire x1="187.96" y1="38.1" x2="190.5" y2="38.1" width="0.1524" layer="91"/>
 <pinref part="SUPPLY18" gate="GND" pin="GND"/>
-<wire x1="185.42" y1="45.72" x2="185.42" y2="43.18" width="0.1524" layer="91"/>
-</segment>
-<segment>
-<pinref part="U2" gate="G$3" pin="CN6_GND"/>
-<wire x1="386.08" y1="0" x2="388.62" y2="0" width="0.1524" layer="91"/>
-<pinref part="SUPPLY26" gate="GND" pin="GND"/>
-<wire x1="388.62" y1="0" x2="388.62" y2="-2.54" width="0.1524" layer="91"/>
+<wire x1="190.5" y1="38.1" x2="190.5" y2="35.56" width="0.1524" layer="91"/>
 </segment>
 </net>
@@
 </segment>
 </net>
-<net name="RESET" class="0">
-<segment>
-<pinref part="U2" gate="G$3" pin="CN6_RESET"/>
-<wire x1="345.44" y1="7.62" x2="340.36" y2="7.62" width="0.1524" layer="91"/>
-<label x="340.36" y="7.62" size="1.778" layer="95" rot="R180" xref="yes"/>
-</segment>
-</net>
-<net name="TP_IRQ" class="0">
-<segment>
-<pinref part="U2" gate="G$4" pin="D3"/>
-<wire x1="261.62" y1="99.06" x2="279.4" y2="99.06" width="0.1524" layer="91"/>
-<label x="279.4" y="99.06" size="1.778" layer="95" xref="yes"/>
-</segment>
-</net>
-<net name="TP_CS" class="0">
-<segment>
-<pinref part="U2" gate="G$4" pin="D4"/>
-<wire x1="261.62" y1="96.52" x2="264.16" y2="96.52" width="0.1524" layer="91"/>
-<label x="264.16" y="96.52" size="1.778" layer="95" xref="yes"/>
-</segment>
-</net>
-<net name="TP_BUSY" class="0">
-<segment>
-<pinref part="U2" gate="G$4" pin="D6"/>
-<wire x1="261.62" y1="91.44" x2="279.4" y2="91.44" width="0.1524" layer="91"/>
-<label x="279.4" y="91.44" size="1.778" layer="95" xref="yes"/>
-</segment>
-</net>
-<net name="LCD_DC" class="0">
-<segment>
-<pinref part="U2" gate="G$4" pin="D7"/>
-<wire x1="261.62" y1="88.9" x2="264.16" y2="88.9" width="0.1524" layer="91"/>
-<label x="264.16" y="88.9" size="1.778" layer="95" xref="yes"/>
-</segment>
-</net>
-<net name="LCD_RST" class="0">
-<segment>
-<pinref part="U2" gate="G$6" pin="D8"/>
-<wire x1="261.62" y1="144.78" x2="279.4" y2="144.78" width="0.1524" layer="91"/>
-<label x="279.4" y="144.78" size="1.778" layer="95" xref="yes"/>
-</segment>
-</net>
-<net name="LCD_BL" class="0">
-<segment>
-<pinref part="U2" gate="G$6" pin="D9"/>
-<wire x1="261.62" y1="142.24" x2="264.16" y2="142.24" width="0.1524" layer="91"/>
-<label x="264.16" y="142.24" size="1.778" layer="95" xref="yes"/>
-</segment>
-</net>
-<net name="LCD_CS" class="0">
-<segment>
-<pinref part="U2" gate="G$6" pin="D10"/>
-<wire x1="261.62" y1="139.7" x2="279.4" y2="139.7" width="0.1524" layer="91"/>
-<label x="279.4" y="139.7" size="1.778" layer="95" xref="yes"/>
-</segment>
-</net>
-<net name="MOSI" class="0">
-<segment>
-<pinref part="U2" gate="G$6" pin="D11"/>
-<wire x1="261.62" y1="137.16" x2="264.16" y2="137.16" width="0.1524" layer="91"/>
-<label x="264.16" y="137.16" size="1.778" layer="95" xref="yes"/>
-</segment>
-</net>
-<net name="MISO" class="0">
-<segment>
-<pinref part="U2" gate="G$6" pin="D12"/>
-<wire x1="261.62" y1="134.62" x2="279.4" y2="134.62" width="0.1524" layer="91"/>
-<label x="279.4" y="134.62" size="1.778" layer="95" xref="yes"/>
-</segment>
-</net>
-<net name="SCLK" class="0">
-<segment>
-<pinref part="U2" gate="G$6" pin="D13"/>
-<wire x1="261.62" y1="132.08" x2="264.16" y2="132.08" width="0.1524" layer="91"/>
-<label x="264.16" y="132.08" size="1.778" layer="95" xref="yes"/>
-</segment>
-</net>
